File: KiCad/eobard/eobard.kicad_sch (KiCad schematic)
At the start: 20 parts, among them J1 UART JACK LEFT, J3 UART Jack Right, SW1 SW_SPST, SW10 SW_SPST, SW11 SW_SPST, SW12 SW_SPST, SW13 SW_SPST, SW14 SW_SPST, SW15 SW_SPST, SW16 SW_SPST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

Commit message: Small Update
Coming back to this to finally finish it :3
Other:
- company: by viniciusbrit -> by primevivian
Changed lines of the file:
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@@
 	(title_block
 		(title "Eobard Split Keyboard")
-		(date "2024-03-25")
+		(date "2024-11-07")
 		(rev "1.3")
-		(company "by viniciusbrit")
+		(company "by primevivian")
 		(comment 4 "This constitutes the design of a single half of a split keyboard.")
 	)
